Commit message: Update rover model URDF

File: src/rover_model/urdf/rover_model.urdf (robot description, URDF)
Before this commit: robot rover_model, 31 links, 30 joints
Links:
- link base_link: geometry collision mesh filename=package://rover_model/meshes/base_link.stl scale=0.001 0.001 0.001; visual mesh filename=package://rover_model/meshes/base_link.stl scale=0.001 0.001 0.001
- link bog1_left: geometry collision mesh filename=package://rover_model/meshes/bog1_left.stl scale=0.001 0.001 0.001; visual mesh filename=package://rover_model/meshes/bog1_left.stl scale=0.001 0.001 0.001
- link bog1_right: geometry collision mesh filename=package://rover_model/meshes/bog1_right.stl scale=0.001 0.001 0.001; visual mesh filename=package://rover_model/meshes/bog1_right.stl scale=0.001 0.001 0.001
- link bog2_left: geometry collision mesh filename=package://rover_model/meshes/bog2_left.stl scale=0.001 0.001 0.001; visual mesh filename=package://rover_model/meshes/bog2_left.stl scale=0.001 0.001 0.001
- link bog2_right: geometry collision mesh filename=package://rover_model/meshes/bog2_right.stl scale=0.001 0.001 0.001; visual mesh filename=package://rover_model/meshes/bog2_right.stl scale=0.001 0.001 0.001
- link bog3_left: geometry collision mesh filename=package://rover_model/meshes/bog3_left.stl scale=0.001 0.001 0.001; visual mesh filename=package://rover_model/meshes/bog3_left.stl scale=0.001 0.001 0.001
- link bog3_right: geometry collision mesh filename=package://rover_model/meshes/bog3_right.stl scale=0.001 0.001 0.001; visual mesh filename=package://rover_model/meshes/bog3_right.stl scale=0.001 0.001 0.001
- link bog_joint_left: geometry collision mesh filename=package://rover_model/meshes/bog_joint_left.stl scale=0.001 0.001 0.001; visual mesh filename=package://rover_model/meshes/bog_joint_left.stl scale=0.001 0.001 0.001
- link bog_joint_right: geometry collision mesh filename=package://rover_model/meshes/bog_joint_right.stl scale=0.001 0.001 0.001; visual mesh filename=package://rover_model/meshes/bog_joint_right.stl scale=0.001 0.001 0.001
- link c_bar_left: geometry collision mesh filename=package://rover_model/meshes/c_bar_left.stl scale=0.001 0.001 0.001; visual mesh filename=package://rover_model/meshes/c_bar_left.stl scale=0.001 0.001 0.001
- link c_bar_right: geometry collision mesh filename=package://rover_model/meshes/c_bar_right.stl scale=0.001 0.001 0.001; visual mesh filename=package://rover_model/meshes/c_bar_right.stl scale=0.001 0.001 0.001
- link camera_link: geometry collision mesh filename=package://rover_model/meshes/camera_link.stl scale=0.001 0.001 0.001; visual mesh filename=package://rover_model/meshes/camera_link.stl scale=0.001 0.001 0.001
- link left_front_wheel_link: geometry collision mesh filename=package://rover_model/meshes/left_front_wheel_link.stl scale=0.001 0.001 0.001; visual mesh filename=package://rover_model/meshes/left_front_wheel_link.stl scale=0.001 0.001 0.001
- link left_mid_wheel_link: geometry collision mesh filename=package://rover_model/meshes/left_mid_wheel_link.stl scale=0.001 0.001 0.001; visual mesh filename=package://rover_model/meshes/left_mid_wheel_link.stl scale=0.001 0.001 0.001
- link left_rear_wheel_link: geometry collision mesh filename=package://rover_model/meshes/left_rear_wheel_link.stl scale=0.001 0.001 0.001; visual mesh filename=package://rover_model/meshes/left_rear_wheel_link.stl scale=0.001 0.001 0.001
- link lidar_link: geometry collision mesh filename=package://rover_model/meshes/lidar_link.stl scale=0.001 0.001 0.001; visual mesh filename=package://rover_model/meshes/lidar_link.stl scale=0.001 0.001 0.001
- link lidar_mount: geometry collision mesh filename=package://rover_model/meshes/lidar_mount.stl scale=0.001 0.001 0.001; visual mesh filename=package://rover_model/meshes/lidar_mount.stl scale=0.001 0.001 0.001
- link main_mount_left: geometry collision mesh filename=package://rover_model/meshes/main_mount_left.stl scale=0.001 0.001 0.001; visual mesh filename=package://rover_model/meshes/main_mount_left.stl scale=0.001 0.001 0.001
- link main_mount_right: geometry collision mesh filename=package://rover_model/meshes/main_mount_right.stl scale=0.001 0.001 0.001; visual mesh filename=package://rover_model/meshes/main_mount_right.stl scale=0.001 0.001 0.001
- link right_front_wheel_link: geometry collision mesh filename=package://rover_model/meshes/right_front_wheel_link.stl scale=0.001 0.001 0.001; visual mesh filename=package://rover_model/meshes/right_front_wheel_link.stl scale=0.001 0.001 0.001
- link right_mid_wheel_link: geometry collision mesh filename=package://rover_model/meshes/right_mid_wheel_link.stl scale=0.001 0.001 0.001; visual mesh filename=package://rover_model/meshes/right_mid_wheel_link.stl scale=0.001 0.001 0.001
- link right_rear_wheel_link: geometry collision mesh filename=package://rover_model/meshes/right_rear_wheel_link.stl scale=0.001 0.001 0.001; visual mesh filename=package://rover_model/meshes/right_rear_wheel_link.stl scale=0.001 0.001 0.001
- link rocker_left: geometry collision mesh filename=package://rover_model/meshes/rocker_left.stl scale=0.001 0.001 0.001; visual mesh filename=package://rover_model/meshes/rocker_left.stl scale=0.001 0.001 0.001
- link rocker_right: geometry collision mesh filename=package://rover_model/meshes/rocker_right.stl scale=0.001 0.001 0.001; visual mesh filename=package://rover_model/meshes/rocker_right.stl scale=0.001 0.001 0.001
- link wheel_joint_1: geometry collision mesh filename=package://rover_model/meshes/wheel_joint_1.stl scale=0.001 0.001 0.001; visual mesh filename=package://rover_model/meshes/wheel_joint_1.stl scale=0.001 0.001 0.001
- link wheel_joint_2: geometry collision mesh filename=package://rover_model/meshes/wheel_joint_2.stl scale=0.001 0.001 0.001; visual mesh filename=package://rover_model/meshes/wheel_joint_2.stl scale=0.001 0.001 0.001
- link wheel_joint_3: geometry collision mesh filename=package://rover_model/meshes/wheel_joint_3.stl scale=0.001 0.001 0.001; visual mesh filename=package://rover_model/meshes/wheel_joint_3.stl scale=0.001 0.001 0.001
- link wheel_joint_4: geometry collision mesh filename=package://rover_model/meshes/wheel_joint_4.stl scale=0.001 0.001 0.001; visual mesh filename=package://rover_model/meshes/wheel_joint_4.stl scale=0.001 0.001 0.001
- link wheel_joint_5: geometry collision mesh filename=package://rover_model/meshes/wheel_joint_5.stl scale=0.001 0.001 0.001; visual mesh filename=package://rover_model/meshes/wheel_joint_5.stl scale=0.001 0.001 0.001
- link wheel_joint_6: geometry collision mesh filename=package://rover_model/meshes/wheel_joint_6.stl scale=0.001 0.001 0.001; visual mesh filename=package://rover_model/meshes/wheel_joint_6.stl scale=0.001 0.001 0.001
